Commit message: moving nose to chassis

File: urdf/car.urdf (robot description, URDF)
Before this commit: robot car, 2 links, 1 joints
Links:
- link chassis: geometry collision mesh filename=file://$(find simulator)/meshes/lrt4/chassis/monocoque.stl scale=${scale} ${scale} ${scale}; visual mesh filename=file://$(find simulator)/meshes/lrt4/chassis/monocoque.stl scale=${scale} ${scale} ${scale}

Commit message: adding motor and cooling jacket

File: urdf/car.urdf (robot description, URDF)
Before this commit: robot car, 2 links, 1 joints
Links:
- link chassis: geometry collision mesh filename=file://$(find simulator)/meshes/lrt4/chassis/monocoque.stl scale=${scale} ${scale} ${scale}; visual mesh filename=file://$(find simulator)/meshes/lrt4/chassis/mono_cfd.stl scale=${scale} ${scale} ${scale}

Commit message: chassis and aero ok, next is VD

File: urdf/car.urdf (robot description, URDF)
Before this commit: robot car, 2 links, 1 joints
Links:
- removed link chassis
